File: hardware/co2warner/co2warner.sch (KiCad schematic (older format))
At the start: 13 parts, among them J1 AVR-ISP-6, U1 ATmega88P-20PU, U2 DHT11, U3 CCS811, U4 HT7733A

Commit message: wire
Connections:
- net at U1.24 (PC1): now also U3.7 (~WAKE)
- no-connect marks 18 -> 16
Changed lines of the file:
@@
 NoConn ~ 2700 2700
 NoConn ~ 2700 2800
-NoConn ~ 2700 3100
 NoConn ~ 2700 3800
 NoConn ~ 2700 3900
@@
 Wire Wire Line
 	9800 2000 10150 2000
-NoConn ~ 6050 4950
 Wire Wire Line
 	10150 1050 10550 1050
+Wire Wire Line
+	6050 4950 4750 4950
+Wire Wire Line
+	4750 4950 4750 3100
+Wire Wire Line
+	4750 3100 2700 3100
 $EndSCHEMATC
